File: hardware/kicad/usb_device.kicad_sch (KiCad schematic)
At the start: 3 parts, among them J2 USB-C_16P-F-SMT

Commit message: fix: repair schematic connectivity, real MAX3421E pinout, footprint assignment
- Root sheet pins were placed outside the sheet boxes, so no cross-sheet
  net (IO5->CI-V, USB D+/D-, SPI, VBUS_5V, 5V_HOST) was actually connected.
  Rebuilt pins on the sheet borders with wire stubs + labels.
- MCU: SW1/SW2 pin 2 carried both GND and EN/BOOT0 (short to ground);
  GND moved to pin 1. Unused ESP32 GPIOs marked no-connect.
- USB_Host rebuilt around the real MAX3421E TQFN-32 pinout (datasheet
  19-3953): 33 ohm D+/D- series resistors, 1uF VCC/VBCOMP, 0.1uF VL.
- J1 now AudioJack3 (T/R/S) with CUI SJ1-3523N footprint; Q1 is a real
  2N7000 (TO-92).
- PWR_FLAGs added; ERC (raw kicad-cli) has 0 errors.
- Board outline 65x45 mm, 54 footprints assigned and written to symbol
  Footprint fields, netlist applied. Placement is a rough grid only; no
  routing yet.
Parts:
- J2: footprint (none) -> Connector_USB:USB_C_Receptacle_GCT_USB4115-03-C
- R8, R9: footprint (none) -> Resistor_SMD:R_0603_1608Metric
Changed lines of the file:
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@@
 			)
 		)
-		(property "Footprint" ""
+		(property "Footprint" "Connector_USB:USB_C_Receptacle_GCT_USB4115-03-C"
 			(at 40 110 0)
 			(effects
@@
 			)
 		)
-		(property "Footprint" ""
+		(property "Footprint" "Resistor_SMD:R_0603_1608Metric"
 			(at 70 100 0)
 			(effects
@@
 			)
 		)
-		(property "Footprint" ""
+		(property "Footprint" "Resistor_SMD:R_0603_1608Metric"
 			(at 70 106 0)
 			(effects
