File: hardware/kicad/rs232_cat.kicad_sch (KiCad schematic)
At the start: 7 parts, among them U4 MAX3232EESE+T

Commit message: Refactor the microcontroller sheet; add switch footprint and 3d file; add titles, date and WaveRig annotation to all sheets.
Other:
- company: (none) -> WaveRig
Changed lines of the file:
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@@
 	(generator_version "10.0")
 	(paper "A4")
+	(title_block
+		(rev "0.1")
+		(company "WaveRig")
+	)
 	(no_connect
 		(at 60.32 117.62)
