File: hardware/kicad/usb_host.kicad_sch (KiCad schematic)
At the start: 10 parts, among them J3 USB-A_Host, U7 MAX3421EETJ+, Y1 12MHz CL18pF ESR60R max

Commit message: Refactor the microcontroller sheet; add switch footprint and 3d file; add titles, date and WaveRig annotation to all sheets.
Other:
- company: (none) -> WaveRig
Changed lines of the file:
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@@
 	(generator_version "10.0")
 	(paper "A4")
+	(title_block
+		(rev "0.1")
+		(company "WaveRig")
+	)
 	(no_connect
 		(at 98.73 127.5)
